File: hardware/sfp2usbc/sfp2usbc.kicad_pcb (KiCad board)
At the start: 4 copper layers, 78 x 50 mm, 24 parts, among them J1 SFP, J2 SFP, J3 USB-C, U1 TPD4E05U06, U2 TPD4E05U06

Commit message: hardware/sfp2usbc: Routed board (route_board.py), DRC clean.
Planned routes generated on the placed board: nested L-shaped 90 ohm pairs with 45 degrees
corners and no crossings (Lane 1 on the top half, Lane 0 on the bottom half as the USB-C pins),
USB-C A row pairs on F.Cu, B row pairs through staggered vias and B.Cu, length matching bumps
(intra-pair skew <= 0.043mm), GND planes/pours/stitching, CC/VBUS/shield.

Netlist: P/N swaps for the crossing-free routing (Lane 1 SFP TD, Lane 0 USB-C TX1: receivers
polarity inversion), ESD lines in the routing order, USB 2.0/VBUS cap/test points removed (VBUS
bottom test pad). Tests: DRC clean and pairs skew on the generated board.

Co-Authored-By: Claude Opus 5.5 <noreply@anthropic.com>
Claude-Session: https://claude.ai/code/session_012xb5QTCQZW5sMRfLG8ccg8
Parts:
- removed C6: 1uF, Capacitor_SMD:C_0402_1005Metric
- removed TP2: CC2, TestPoint:TestPoint_Pad_D1.0mm
- removed TP3: VBUS, TestPoint:TestPoint_Pad_D1.0mm
- removed TP4: USB2_DP, TestPoint:TestPoint_Pad_D1.0mm
- removed TP5: USB2_DN, TestPoint:TestPoint_Pad_D1.0mm
- removed TP6: GND, TestPoint:TestPoint_Pad_D1.0mm
- TP1: value CC1 -> VBUS; moved to B.Cu
- moved C4 23.2 mm to (147.5, 116.6)
- moved C1 23.1 mm to (145.5, 137.8)
- moved TP1 22.1 mm to (173.0, 125.2)
- moved J1 22.0 mm to (143.0, 136.0)
- moved J2 22.0 mm to (143.0, 114.0)
- moved C3 21.5 mm to (145.5, 115.8)
- moved C2 20.9 mm to (147.5, 138.6)
- moved U1 11.8 mm to (161.5, 129.8)
- moved U2 11.1 mm to (161.5, 121.0)
- moved C5 3.76 mm to (171.6, 132.6), turned to -90 degrees
- moved R1 3.55 mm to (164.6, 125.8), turned to 180 degrees
- moved R2 3.30 mm to (164.6, 124.5), turned to 180 degrees
- moved R3 0.60 mm to (170.0, 132.6), turned to -90 degrees
Connections:
- J2 pad 18: /L1_SSRX_P -> /L1_SSRX_N
- J2 pad 19: /L1_SSRX_N -> /L1_SSRX_P
- J3 pad A2: /L0_SSTX_P -> /L0_SSTX_N
- J3 pad A3: /L0_SSTX_N -> /L0_SSTX_P
- J3 pad A6: /USB2_DP -> (no net)
- J3 pad A7: /USB2_DN -> (no net)
- J3 pad B6: /USB2_DP -> (no net)
- J3 pad B7: /USB2_DN -> (no net)
- TP1 pad 1: /CC1 -> /VBUS
- U1 pad 1: /L0_SSTX_P -> /L0_SSRX_N
- U1 pad 10: /L0_SSTX_P -> /L0_SSRX_N
- U1 pad 2: /L0_SSTX_N -> /L0_SSRX_P
- U1 pad 4: /L0_SSRX_P -> /L0_SSTX_P
- U1 pad 5: /L0_SSRX_N -> /L0_SSTX_N
- U1 pad 6: /L0_SSRX_N -> /L0_SSTX_N
- U1 pad 7: /L0_SSRX_P -> /L0_SSTX_P
- U1 pad 9: /L0_SSTX_N -> /L0_SSRX_P
- U2 pad 1: /L1_SSTX_P -> /L1_SSRX_P
- U2 pad 10: /L1_SSTX_P -> /L1_SSRX_P
- U2 pad 2: /L1_SSTX_N -> /L1_SSRX_N
- U2 pad 4: /L1_SSRX_P -> /L1_SSTX_P
- U2 pad 5: /L1_SSRX_N -> /L1_SSTX_N
- U2 pad 6: /L1_SSRX_N -> /L1_SSTX_N
- U2 pad 7: /L1_SSRX_P -> /L1_SSTX_P
- U2 pad 9: /L1_SSTX_N -> /L1_SSRX_N
Routing:
- net /L0_SSRX_N: track 0.00 -> 36.1 mm, vias 0 -> 2
- net /L0_SSRX_P: track 0.00 -> 36.0 mm, vias 0 -> 2
- net /L1_SSRX_P: track 0.00 -> 36.0 mm
- net /L1_SSRX_N: track 0.00 -> 36.0 mm
- net /L1_SSTX_P: track 0.00 -> 32.0 mm, vias 0 -> 2
- net /L1_SSTX_N: track 0.00 -> 30.0 mm, vias 0 -> 2
- net /L0_SSTX_P: track 0.00 -> 30.0 mm
- net /L0_SSTX_N: track 0.00 -> 28.0 mm
- net /GND: track 0.00 -> 25.9 mm, vias 0 -> 334
- net /SHIELD: track 0.00 -> 25.5 mm
- net /VBUS: track 0.00 -> 10.1 mm, vias 0 -> 2
- net /CC2: track 0.00 -> 6.61 mm, vias 0 -> 2
- net /L1_SFP_RD_N: track 0.00 -> 6.12 mm
- net /L0_SFP_RD_N: track 0.00 -> 6.12 mm
- net /L1_SFP_RD_P: track 0.00 -> 4.12 mm
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- added copper zone on B.Cu, net /GND
- added copper zone on F.Cu, net /GND
- added copper zone on In1.Cu, net /GND
- added copper zone on In2.Cu, net /GND
