File: hardware/sfp2usbc/sfp2usbc.kicad_sch (KiCad schematic)
At the start: 24 parts, among them J1 SFP, J2 SFP, J3 USB-C, U1 TPD4E05U06, U2 TPD4E05U06

Commit message: hardware/sfp2usbc: Routed board (route_board.py), DRC clean.
Planned routes generated on the placed board: nested L-shaped 90 ohm pairs with 45 degrees
corners and no crossings (Lane 1 on the top half, Lane 0 on the bottom half as the USB-C pins),
USB-C A row pairs on F.Cu, B row pairs through staggered vias and B.Cu, length matching bumps
(intra-pair skew <= 0.043mm), GND planes/pours/stitching, CC/VBUS/shield.

Netlist: P/N swaps for the crossing-free routing (Lane 1 SFP TD, Lane 0 USB-C TX1: receivers
polarity inversion), ESD lines in the routing order, USB 2.0/VBUS cap/test points removed (VBUS
bottom test pad). Tests: DRC clean and pairs skew on the generated board.

Co-Authored-By: Claude Opus 5.5 <noreply@anthropic.com>
Claude-Session: https://claude.ai/code/session_012xb5QTCQZW5sMRfLG8ccg8
Parts:
- removed C6: 1uF, Capacitor_SMD:C_0402_1005Metric, symbol Device:C
- removed TP2: CC2, TestPoint:TestPoint_Pad_D1.0mm, symbol Connector:TestPoint
- removed TP3: VBUS, TestPoint:TestPoint_Pad_D1.0mm, symbol Connector:TestPoint
- removed TP4: USB2_DP, TestPoint:TestPoint_Pad_D1.0mm, symbol Connector:TestPoint
- removed TP5: USB2_DN, TestPoint:TestPoint_Pad_D1.0mm, symbol Connector:TestPoint
- removed TP6: GND, TestPoint:TestPoint_Pad_D1.0mm, symbol Connector:TestPoint
- TP1: value CC1 -> VBUS
Connections:
- net CC1: no longer TP1.1
- net L0_SSRX_N: now also U1.1 (D1+), U1.10 (NC); no longer U1.5 (D2-), U1.6 (NC)
- net L0_SSRX_P: now also U1.2 (D1-), U1.9 (NC); no longer U1.4 (D2+), U1.7 (NC)
- net L0_SSTX_N: now also J3.A2 (TX1+), U1.5 (D2-), U1.6 (NC); no longer J3.A3 (TX1-), U1.2 (D1-), U1.9 (NC)
- net L0_SSTX_P: now also J3.A3 (TX1-), U1.4 (D2+), U1.7 (NC); no longer J3.A2 (TX1+), U1.1 (D1+), U1.10 (NC)
- net L1_SSRX_N: now also J2.18 (TD+), U2.2 (D1-), U2.9 (NC); no longer J2.19 (TD-), U2.5 (D2-), U2.6 (NC)
- net L1_SSRX_P: now also J2.19 (TD-), U2.1 (D1+), U2.10 (NC); no longer J2.18 (TD+), U2.4 (D2+), U2.7 (NC)
- net L1_SSTX_N: now also U2.5 (D2-), U2.6 (NC); no longer U2.2 (D1-), U2.9 (NC)
- net L1_SSTX_P: now also U2.4 (D2+), U2.7 (NC); no longer U2.1 (D1+), U2.10 (NC)
- net VBUS: now also TP1.1
- net USB2_DN: no longer names the net of J3.A7 (D-)
- net USB2_DN: no longer J3.B7 (D-)
- net USB2_DP: no longer names the net of J3.A6 (D+)
- net USB2_DP: no longer J3.B6 (D+)
- no-connect marks 22 -> 26
Other:
- note added: "Power flag"
- note added: "Rd (UFP), VBUS test pad, shield"
- note removed: "Rd (UFP), VBUS, shield"
- note removed: "Test points, power flag"
- moved on the sheet: TP1
